Commit message: exercise: Add the robot wheels as links and connect these to the chassis using joints

File: urdf/udacity_bot.xacro (robot description, xacro)
@@ -55,3 +55,65 @@
 		</visual>
 	</link>
+	<link name="left_wheel">
+		<inertial>
+			<mass value="5"/>
+			<origin xyz="0 0 0" rpy="0 1.5707 1.5707"/>
+			<inertia
+				ixx="0.1" ixy="0" ixz="0"
+				iyy="0.1" iyz="0"
+				izz="0.1"
+			/>
+		</inertial>
+		<collision>
+			<origin xyz="0 0 0" rpy="0 1.5707 1.5707"/>
+			<geometry>
+				<cylinder radius="0.1" length="0.05"/>
+			</geometry>
+		</collision>
+		<visual>
+			<origin xyz="0 0 0" rpy="0 1.5707 1.5707"/>
+			<geometry>
+				<cylinder radius="0.1" length="0.05"/>
+			</geometry>
+		</visual>
+	</link>
+	<link name="right_wheel">
+		<inertial>
+			<mass value="5"/>
+			<origin xyz="0 0 0" rpy="0 1.5707 1.5707"/>
+			<inertia
+				ixx="0.1" ixy="0" ixz="0"
+				iyy="0.1" iyz="0"
+				izz="0.1"
+			/>
+		</inertial>
+		<collision>
+			<origin xyz="0 0 0" rpy="0 1.5707 1.5707"/>
+			<geometry>
+				<cylinder radius="0.1" length="0.05"/>
+			</geometry>
+		</collision>
+		<visual>
+			<origin xyz="0 0 0" rpy="0 1.5707 1.5707"/>
+			<geometry>
+				<cylinder radius="0.1" length="0.05"/>
+			</geometry>
+		</visual>
+	</link>
+	<joint type="continuous" name="left_wheel_hinge">
+		<origin xyz="0 0.15 0" rpy="0 0 0"/>
+		<child link="left_wheel"/>
+		<parent link="chassis"/>
+		<axis xyz="0 1 0" rpy="0 0 0"/>
+		<limit effort="10000" velocity="1000"/>
+		<dynamics damping="1.0" friction="1.0"/>
+	</joint>
+	<joint type="continuous" name="right_wheel_hinge">
+		<origin xyz="0 -0.15 0" rpy="0 0 0"/>
+		<child link="right_wheel"/>
+		<parent link="chassis"/>
+		<axis xyz="0 1 0" rpy="0 0 0"/>
+		<limit effort="10000" velocity="1000"/>
+		<dynamics damping="1.0" friction="1.0"/>
+	</joint>
 </robot>

Commit message: exercise: Added camera sensor to the robot chassis

File: urdf/udacity_bot.xacro (robot description, xacro)
@@ -117,3 +117,31 @@
 		<dynamics damping="1.0" friction="1.0"/>
 	</joint>
+	<link name="camera">
+		<inertial>
+			<mass value="0.1"/>
+			<origin xyz="0 0 0" rpy="0 0 0"/>
+			<inertia
+				ixx="1e-6" ixy="0" ixz="0"
+				iyy="1e-6" iyz="0"
+				izz="1e-6"
+			/>
+		</inertial>
+		<collision>
+			<origin xyz="" rpy=""/>
+			<geometry>
+				<box size="0.05"/>
+			</geometry>
+		</collision>
+		<visual>
+			<origin xyz="" rpy=""/>
+			<geometry>
+				<box size="0.05"/>
+			</geometry>
+		</visual>
+	</link>
+	<joint type="continuous" name="camera_joint">
+		<origin xyz="0.2 0 0" rpy="0 0 0"/>
+		<parent link="chassis"/>
+		<child link="camera"/>
+	</joint>
 </robot>

Commit message: exercise: Changed joint type from continuous to fixed - camera does not move

File: urdf/udacity_bot.xacro (robot description, xacro)
@@ -140,5 +140,5 @@
 		</visual>
 	</link>
-	<joint type="continuous" name="camera_joint">
+	<joint type="fixed" name="camera_joint">
 		<origin xyz="0.2 0 0" rpy="0 0 0"/>
 		<parent link="chassis"/>

Commit message: exercise: Updated the robot xacro file to include the camera and laser rangefinder sensors

File: urdf/udacity_bot.xacro (robot description, xacro)
@@ -1,5 +1,7 @@
 <?xml version='1.0'?>
 <robot name="udacity_bot" xmlns:xacro="http://www.ros.org/wiki/xacro">
+	<!-- Not sure what this part is -->
 	<link name="robot_footprint"></link>
+	<!-- Joint from robot footprint to chassis -->
 	<joint name="robot_footprint_joint" type="fixed">
 		<origin xyz="0 0 0" rpy="0 0 0" />
@@ -7,4 +9,5 @@
 		<child link="chassis" />
 	</joint>
+	<!-- The robot chassis -->
 	<link name="chassis">
 		<pose>0 0 0.1 0 0 0</pose>
@@ -55,4 +58,5 @@
 		</visual>
 	</link>
+	<!-- Robot left wheel -->
 	<link name="left_wheel">
 		<inertial>
@@ -78,4 +82,5 @@
 		</visual>
 	</link>
+	<!-- Robot right wheel -->
 	<link name="right_wheel">
 		<inertial>
@@ -101,4 +106,5 @@
 		</visual>
 	</link>
+	<!-- Joint connecting the left wheel to the chassis -->
 	<joint type="continuous" name="left_wheel_hinge">
 		<origin xyz="0 0.15 0" rpy="0 0 0"/>
@@ -109,4 +115,5 @@
 		<dynamics damping="1.0" friction="1.0"/>
 	</joint>
+	<!-- Joint connecting the right wheel to the chassis -->
 	<joint type="continuous" name="right_wheel_hinge">
 		<origin xyz="0 -0.15 0" rpy="0 0 0"/>
@@ -117,4 +124,5 @@
 		<dynamics damping="1.0" friction="1.0"/>
 	</joint>
+	<!-- Camera -->
 	<link name="camera">
 		<inertial>
@@ -140,4 +148,5 @@
 		</visual>
 	</link>
+	<!-- Joint connecting the camera to the chassis -->
 	<joint type="fixed" name="camera_joint">
 		<origin xyz="0.2 0 0" rpy="0 0 0"/>
@@ -145,3 +154,33 @@
 		<child link="camera"/>
 	</joint>
+	<!-- Laser Range Finder -->
+	<link name="hokuyo">
+		<inertial>
+			<mass value="0.1"/>
+			<origin xyz="0 0 0" rpy="0 0 0"/>
+			<inertia
+				ixx="1e-6" ixy="0" ixz="0"
+				iyy="1e-6" iyz="0"
+				izz="1e-6"
+			/>
+		</inertial>
+		<collision>
+			<origin xyz="0 0 0" rpy="0 0 0"/>
+			<geometry>
+				<box size="0.1"/>
+			</geometry>
+		</collision>
+		<visual>
+			<origin xyz="0 0 0" rpy="0 0 0"/>
+			<geometry>
+				<mesh filename="package://udacity_bot/meshes/hokuyo.dae"/>
+			</geometry>
+		</visual>
+	</link>
+	<!-- Joint connecting the  -->
+	<joint type="fixed" name="hokuyo_joint">
+		<origin xyz="0.15 0 0.1" rpy="0 0 0"/>
+		<parent link="chassis"/>
+		<child link="hokuyo"/>
+	</joint>
 </robot>

Commit message: exercise: Added the origin xyz and rpy to the collision and visual tags

File: urdf/udacity_bot.xacro (robot description, xacro)
@@ -138,5 +138,5 @@
 		</inertial>
 		<collision>
-			<origin xyz="" rpy=""/>
+			<origin xyz="0 0 0" rpy="0 0 0"/>
 			<geometry>
 				<box size="0.05"/>
@@ -144,5 +144,5 @@
 		</collision>
 		<visual>
-			<origin xyz="" rpy=""/>
+			<origin xyz="0 0 0" rpy="0 0 0"/>
 			<geometry>
 				<box size="0.05"/>

Commit message: exercise: Corrected the box dimensions - three box dimensions are always needed

File: urdf/udacity_bot.xacro (robot description, xacro)
@@ -140,5 +140,5 @@
 			<origin xyz="0 0 0" rpy="0 0 0"/>
 			<geometry>
-				<box size="0.05"/>
+				<box size="0.05 0.05 0.05"/>
 			</geometry>
 		</collision>
@@ -170,5 +170,5 @@
 			<origin xyz="0 0 0" rpy="0 0 0"/>
 			<geometry>
-				<box size="0.1"/>
+				<box size="0.1 0.1 0.1"/>
 			</geometry>
 		</collision>

Commit message: exercise: final correction to the camera (the visual box dimensions were missing)

File: urdf/udacity_bot.xacro (robot description, xacro)
@@ -146,5 +146,5 @@
 			<origin xyz="0 0 0" rpy="0 0 0"/>
 			<geometry>
-				<box size="0.05"/>
+				<box size="0.05 0.05 0.05"/>
 			</geometry>
 		</visual>

Commit message: exercise: Add colour changes to the visual properties of the chassis, wheels and camera

File: urdf/udacity_bot.xacro (robot description, xacro)
@@ -30,4 +30,5 @@
 		</collision>
 		<visual name="chassis_visual">
+			<material name="blue"/>
 			<origin xyz="0 0 0" rpy="0 0 0"/>
 			<geometry>
@@ -78,4 +79,5 @@
 		</collision>
 		<visual>
+			<material name="green"/>
 			<origin xyz="0 0 0" rpy="0 1.5707 1.5707"/>
 			<geometry>
@@ -102,4 +104,5 @@
 		</collision>
 		<visual>
+			<material name="green"/>
 			<origin xyz="0 0 0" rpy="0 1.5707 1.5707"/>
 			<geometry>
@@ -144,4 +147,5 @@
 		</collision>
 		<visual>
+			<material name="red"/>
 			<origin xyz="0 0 0" rpy="0 0 0"/>
 			<geometry>

Commit message: exercise: changed the location of the material tags (need to be outside of the visual tag)

File: urdf/udacity_bot.xacro (robot description, xacro)
@@ -13,4 +13,5 @@
 	<!-- The robot chassis -->
 	<link name="chassis">
+		<material name="blue"/>
 		<pose>0 0 0.1 0 0 0</pose>
 		<inertial>
@@ -30,5 +31,4 @@
 		</collision>
 		<visual name="chassis_visual">
-			<material name="blue"/>
 			<origin xyz="0 0 0" rpy="0 0 0"/>
 			<geometry>
@@ -63,4 +63,5 @@
 	<!-- Robot left wheel -->
 	<link name="left_wheel">
+		<material name="green"/>
 		<inertial>
 			<mass value="5"/>
@@ -79,5 +80,4 @@
 		</collision>
 		<visual>
-			<material name="green"/>
 			<origin xyz="0 0 0" rpy="0 1.5707 1.5707"/>
 			<geometry>
@@ -88,4 +88,5 @@
 	<!-- Robot right wheel -->
 	<link name="right_wheel">
+		<material name="green"/>
 		<inertial>
 			<mass value="5"/>
@@ -104,5 +105,4 @@
 		</collision>
 		<visual>
-			<material name="green"/>
 			<origin xyz="0 0 0" rpy="0 1.5707 1.5707"/>
 			<geometry>
@@ -131,4 +131,5 @@
 	<!-- Camera -->
 	<link name="camera">
+		<material name="red"/>
 		<inertial>
 			<mass value="0.1"/>
@@ -147,5 +148,4 @@
 		</collision>
 		<visual>
-			<material name="red"/>
 			<origin xyz="0 0 0" rpy="0 0 0"/>
 			<geometry>

Commit message: Revert "exercise: Add colour changes to the visual properties of the chassis, wheels and camera"
This reverts commit a13e46aab543d6cbfb2a1eef7fddfa4bd3a8651d.

File: urdf/udacity_bot.xacro (robot description, xacro)
@@ -13,5 +13,4 @@
 	<!-- The robot chassis -->
 	<link name="chassis">
-		<material name="blue"/>
 		<pose>0 0 0.1 0 0 0</pose>
 		<inertial>
@@ -35,4 +34,5 @@
 				<box size="0.4 0.2 0.1"/>
 			</geometry>
+			<material name="blue"/>
 		</visual>
 		<collision name='back_caster_collision'>
@@ -63,5 +63,4 @@
 	<!-- Robot left wheel -->
 	<link name="left_wheel">
-		<material name="green"/>
 		<inertial>
 			<mass value="5"/>
@@ -84,9 +83,9 @@
 				<cylinder radius="0.1" length="0.05"/>
 			</geometry>
+			<material name="green"/>
 		</visual>
 	</link>
 	<!-- Robot right wheel -->
 	<link name="right_wheel">
-		<material name="green"/>
 		<inertial>
 			<mass value="5"/>
@@ -109,4 +108,5 @@
 				<cylinder radius="0.1" length="0.05"/>
 			</geometry>
+			<material name="green"/>
 		</visual>
 	</link>
@@ -131,5 +131,4 @@
 	<!-- Camera -->
 	<link name="camera">
-		<material name="red"/>
 		<inertial>
 			<mass value="0.1"/>
@@ -152,4 +151,5 @@
 				<box size="0.05 0.05 0.05"/>
 			</geometry>
+			<material name="red"/>
 		</visual>
 	</link>

Commit message: Update: change to the robot model

File: urdf/udacity_bot.xacro (robot description, xacro)
@@ -25,5 +25,5 @@
 			/>
 		</inertial>
-		<collision name='collision'>
+		<collision name="chassis_collision">
 			<origin xyz="0 0 0" rpy="0 0 0"/>
 			<geometry>
